Commit message: multi_ns_gazebo

File: urdf/2f_85.ros2_control.xacro (robot description, xacro)
@@ -18,5 +18,5 @@
         gripper_max_force:=235.0
         gripper_closed_position:=0.7929">
-        <ros2_control name="${name}" type="system">
+        <ros2_control name="${prefix + name}" type="system">
             <!-- Plugins -->
             <!--xacro:unless value="${robot and sim_ignition}"-->

File: urdf/fr3_robotiq.urdf.xacro (robot description, xacro)
@@ -1,4 +1,4 @@
 <?xml version='1.0' encoding='utf-8'?>
-<robot xmlns:xacro="http://www.ros.org/wiki/xacro" name="fr3">
+<robot xmlns:xacro="http://www.ros.org/wiki/xacro" name="$(arg arm_prefix)fr3">
   <xacro:include filename="$(find franka_robotiq)/urdf/franka_robotiq.xacro"/>
   <!--
@@ -10,4 +10,6 @@
   <!-- Don't print a prefix for joints, visuals, and links? -->
   <xacro:arg name="no_prefix" default="false"/>
+  <!-- Prefix for joints, visuals, and links -->
+  <xacro:arg name="arm_prefix" default=""/>
   <!-- Should an end-effector be mounted at the flange?" -->
   <xacro:arg name="hand" default="true" />
@@ -30,6 +32,12 @@
   <!-- For a multi arm setup, we need a threaded robot running async-->
   <xacro:arg name="multi_arm" default="false" />
+  <!-- For a multi arm setup, we need a threaded robot running async-->
+  <xacro:arg name="ns" default="" />
+  <!-- Position and orientation with respect to the base -->
+  <xacro:arg name="xyz" default="0 0 0" />
+  <xacro:arg name="rpy" default="0 0 0" />
   <!-- Port for gripper communication-->
   <xacro:arg name="com_port" default='/dev/ttyUSB0' />
+  <xacro:arg name="index" default='0' />
   <xacro:franka_robotiq arm_id="$(arg arm_id)"
                       joint_limits="${xacro.load_yaml('$(find franka_description)/robots/fr3/joint_limits.yaml')}"
@@ -47,6 +55,10 @@
                       gazebo_effort="$(arg gazebo_effort)"
                       no_prefix="$(arg no_prefix)"
-                      arm_prefix= ""
-                      connected_to= "base">
+                      arm_prefix= "$(arg arm_prefix)"
+                      connected_to= "base"
+                      index="$(arg index)"
+                      xyz="$(arg xyz)"
+                      rpy="$(arg rpy)"
+                      ns="$(arg ns)">
   </xacro:franka_robotiq>
 </robot>

File: urdf/franka_arm.ros2_control.xacro (robot description, xacro)
@@ -12,4 +12,6 @@
              multi_arm:=false
              ee_id:=''
+             index:='0'
+             ns:=''
              gripper_closed_position:=0.7929">
     <xacro:property name="arm_prefix_modified" value="${'' if arm_prefix == '' else arm_prefix + '_'}" />
@@ -24,5 +26,5 @@
           </xacro:if>
           <xacro:if value="${gazebo}">
-            <plugin>ign_ros2_control/IgnitionSystem</plugin>
+            <plugin>gz_ros2_control/GazeboSimSystem</plugin>
           </xacro:if>
           <xacro:if value="${use_fake_hardware == 0 and gazebo == 0 and multi_arm == 0}">
@@ -37,9 +39,4 @@
           </xacro:if>
         </hardware>
-        <!--xacro:if value="${gazebo and hand and ee_id == 'robotiq'}">
-          <hardware>
-            <plugin>ign_ros2_control/IgnitionSystem</plugin>
-          </hardware>
-        </xacro:if-->
       <xacro:macro name="configure_joint" params="joint_name initial_position">
         <joint name="${joint_name}">
@@ -48,5 +45,5 @@
             https://github.com/ros-controls/gz_ros2_control/issues/343
             Command Interfaces -->
-          <xacro:if value="${multi_arm == 0}">
+          <xacro:if value="${multi_arm == 0 or gazebo == 1 or use_fake_hardware == 1}">
             <command_interface name="position"/>
             <command_interface name="velocity"/>
@@ -138,17 +135,26 @@
     </ros2_control>
     <xacro:if value="${gazebo}">
-      <gazebo>
-        <plugin filename="ign_ros2_control-system" name="ign_ros2_control::IgnitionROS2ControlPlugin">
-          <parameters>$(find franka_gazebo_bringup)/config/franka_gazebo_controllers.yaml</parameters>
-        </plugin>
-      </gazebo>
+      <xacro:unless value="${multi_arm}">
+        <gazebo>
+          <plugin filename="gz_ros2_control-system" name="gz_ros2_control::GazeboSimROS2ControlPlugin">
+            <!--parameters>$(find franka_robotiq)/config/franka_gazebo_controllers.yaml</parameters-->
+            <!--parameters>$(find franka_bringup)/config/controllers.yaml</parameters-->
+            <parameters>$(find franka_robotiq)/config/${arm_prefix}_controllers.yaml</parameters>
+            <!--controller_manager_prefix_node_name>${ns}/</controller_manager_prefix_node_name-->
+            <ros>
+              <namespace>${ns}</namespace>
+            </ros>
+            <!--robot_param>robot_description</robot_param-->
+          </plugin>
+        </gazebo>
+      </xacro:unless>
+      <xacro:if value="${multi_arm==1 and index=='0'}">
+        <gazebo>
+          <plugin filename="ign_ros2_control-system" name="ign_ros2_control::IgnitionROS2ControlPlugin">
+            <parameters>$(find franka_robotiq)/config/multi_franka_gazebo_controllers.yaml</parameters>
+          </plugin>
+        </gazebo>
+      </xacro:if>
     </xacro:if>
-    <!--xacro:if value="${gazebo and hand and ee_id == 'robotiq'}">
-      <gazebo>
-        <plugin filename="ign_ros2_control-system" name="ign_ros2_control::IgnitionROS2ControlPlugin">
-          <parameters>$(find robotiq_description)/config/robotiq_controllers.yaml</parameters>
-        </plugin>
-      </gazebo>
-    </xacro:if-->
   </xacro:macro>
 </robot>

File: urdf/franka_robotiq.xacro (robot description, xacro)
@@ -23,7 +23,9 @@
                       connected_to:='base'
                       multi_arm:=false
+                      index:='0'
+                      ns:=''
                       com_port:='/dev/ttyUSB0'" >
     <xacro:include filename="$(find franka_description)/robots/common/utils.xacro" />
-    <xacro:include filename="$(find franka_description)/robots/common/franka_arm.xacro" />
+    <xacro:include filename="$(find franka_robotiq)/urdf/franka_arm.xacro" />
     <xacro:property name="arm_prefix_modified" value="${'' if arm_prefix == '' else arm_prefix + '_'}" />
     <xacro:franka_arm
@@ -75,5 +77,5 @@
       <!--xacro:include filename="$(find franka_description)/end_effectors/$(arg ee_id)/$(arg ee_id)_arguments.xacro" /-->
       <xacro:property name="ee_color" value="black" />
-      <xacro:property name="connection" value="${arm_id + '_link8'}" />
+      <xacro:property name="connection" value="${arm_prefix_modified + arm_id + '_link8'}" />
       <xacro:robotiq_gripper name="RobotiqGripperHardwareInterface" prefix="${arm_prefix_modified}" parent="${connection}" use_fake_hardware="$(arg use_fake_hardware)" com_port="$(arg com_port)" sim_ignition="${gazebo}" robot="true">
         <origin xyz="0 0 0" rpy="0 0 0" />
@@ -85,5 +87,5 @@
       <xacro:include filename="$(find franka_description)/end_effectors/$(arg ee_id)/$(arg ee_id)_arguments.xacro" />
       <xacro:property name="special_connection" value="$(arg special_connection)" />
-      <xacro:property name="connection" value="${special_connection if special_connection == '' else arm_id + '_link8'}" />
+      <xacro:property name="connection" value="${special_connection if special_connection == '' else arm_prefix_modified + arm_id + '_link8'}" />
       <xacro:ee_with_one_link
         connected_to="${arm_prefix_modified}${connection}"
@@ -103,5 +105,5 @@
     </xacro:if>
     <!-- Definition of additional Gazebo tags -->
-    <xacro:if value="${gazebo}">
+    <xacro:if value="${gazebo and not multi_arm}">
       <xacro:if value="${parent != ''}">
         <!-- Gazebo requires a joint to a link called "world" for statically mounted robots -->
@@ -112,32 +114,39 @@
           <origin xyz="${xyz}" rpy="${rpy}" />
           <parent link="${parent}" />
-          <child  link="${arm_id}_link0" />
+          <child  link="${arm_prefix_modified}${arm_id}_link0" />
         </joint>
       </xacro:if>
-      <xacro:gazebo-joint joint="${arm_id}_joint1" transmission="hardware_interface/PositionJointInterface" />
-      <xacro:gazebo-joint joint="${arm_id}_joint2" transmission="hardware_interface/PositionJointInterface" />
-      <xacro:gazebo-joint joint="${arm_id}_joint3" transmission="hardware_interface/PositionJointInterface" />
-      <xacro:gazebo-joint joint="${arm_id}_joint4" transmission="hardware_interface/PositionJointInterface" />
-      <xacro:gazebo-joint joint="${arm_id}_joint5" transmission="hardware_interface/PositionJointInterface" />
-      <xacro:gazebo-joint joint="${arm_id}_joint6" transmission="hardware_interface/PositionJointInterface" />
-      <xacro:gazebo-joint joint="${arm_id}_joint7" transmission="hardware_interface/PositionJointInterface" />
-      <xacro:gazebo-joint joint="${arm_id}_joint1" transmission="hardware_interface/VelocityJointInterface" />
-      <xacro:gazebo-joint joint="${arm_id}_joint2" transmission="hardware_interface/VelocityJointInterface" />
-      <xacro:gazebo-joint joint="${arm_id}_joint3" transmission="hardware_interface/VelocityJointInterface" />
-      <xacro:gazebo-joint joint="${arm_id}_joint4" transmission="hardware_interface/VelocityJointInterface" />
-      <xacro:gazebo-joint joint="${arm_id}_joint5" transmission="hardware_interface/VelocityJointInterface" />
-      <xacro:gazebo-joint joint="${arm_id}_joint6" transmission="hardware_interface/VelocityJointInterface" />
-      <xacro:gazebo-joint joint="${arm_id}_joint7" transmission="hardware_interface/VelocityJointInterface" />
-      <xacro:gazebo-joint joint="${arm_id}_joint1" transmission="hardware_interface/EffortJointInterface" />
-      <xacro:gazebo-joint joint="${arm_id}_joint2" transmission="hardware_interface/EffortJointInterface" />
-      <xacro:gazebo-joint joint="${arm_id}_joint3" transmission="hardware_interface/EffortJointInterface" />
-      <xacro:gazebo-joint joint="${arm_id}_joint4" transmission="hardware_interface/EffortJointInterface" />
-      <xacro:gazebo-joint joint="${arm_id}_joint5" transmission="hardware_interface/EffortJointInterface" />
-      <xacro:gazebo-joint joint="${arm_id}_joint6" transmission="hardware_interface/EffortJointInterface" />
-      <xacro:gazebo-joint joint="${arm_id}_joint7" transmission="hardware_interface/EffortJointInterface" />
+      <!--xacro:if value="${gazebo and multi_arm}">
+        <joint name="${connected_to}_link0_joint" type="fixed">
+          <parent link="${connected_to}"/>
+          <child link="${arm_prefix_modified}${arm_id}_link0"/>
+          <origin rpy="${rpy}" xyz="${xyz}"/>
+        </joint>
+      </xacro:if-->
+      <xacro:gazebo-joint joint="${arm_prefix_modified}${arm_id}_joint1" transmission="hardware_interface/PositionJointInterface" />
+      <xacro:gazebo-joint joint="${arm_prefix_modified}${arm_id}_joint2" transmission="hardware_interface/PositionJointInterface" />
+      <xacro:gazebo-joint joint="${arm_prefix_modified}${arm_id}_joint3" transmission="hardware_interface/PositionJointInterface" />
+      <xacro:gazebo-joint joint="${arm_prefix_modified}${arm_id}_joint4" transmission="hardware_interface/PositionJointInterface" />
+      <xacro:gazebo-joint joint="${arm_prefix_modified}${arm_id}_joint5" transmission="hardware_interface/PositionJointInterface" />
+      <xacro:gazebo-joint joint="${arm_prefix_modified}${arm_id}_joint6" transmission="hardware_interface/PositionJointInterface" />
+      <xacro:gazebo-joint joint="${arm_prefix_modified}${arm_id}_joint7" transmission="hardware_interface/PositionJointInterface" />
+      <xacro:gazebo-joint joint="${arm_prefix_modified}${arm_id}_joint1" transmission="hardware_interface/VelocityJointInterface" />
+      <xacro:gazebo-joint joint="${arm_prefix_modified}${arm_id}_joint2" transmission="hardware_interface/VelocityJointInterface" />
+      <xacro:gazebo-joint joint="${arm_prefix_modified}${arm_id}_joint3" transmission="hardware_interface/VelocityJointInterface" />
+      <xacro:gazebo-joint joint="${arm_prefix_modified}${arm_id}_joint4" transmission="hardware_interface/VelocityJointInterface" />
+      <xacro:gazebo-joint joint="${arm_prefix_modified}${arm_id}_joint5" transmission="hardware_interface/VelocityJointInterface" />
+      <xacro:gazebo-joint joint="${arm_prefix_modified}${arm_id}_joint6" transmission="hardware_interface/VelocityJointInterface" />
+      <xacro:gazebo-joint joint="${arm_prefix_modified}${arm_id}_joint7" transmission="hardware_interface/VelocityJointInterface" />
+      <xacro:gazebo-joint joint="${arm_prefix_modified}${arm_id}_joint1" transmission="hardware_interface/EffortJointInterface" />
+      <xacro:gazebo-joint joint="${arm_prefix_modified}${arm_id}_joint2" transmission="hardware_interface/EffortJointInterface" />
+      <xacro:gazebo-joint joint="${arm_prefix_modified}${arm_id}_joint3" transmission="hardware_interface/EffortJointInterface" />
+      <xacro:gazebo-joint joint="${arm_prefix_modified}${arm_id}_joint4" transmission="hardware_interface/EffortJointInterface" />
+      <xacro:gazebo-joint joint="${arm_prefix_modified}${arm_id}_joint5" transmission="hardware_interface/EffortJointInterface" />
+      <xacro:gazebo-joint joint="${arm_prefix_modified}${arm_id}_joint6" transmission="hardware_interface/EffortJointInterface" />
+      <xacro:gazebo-joint joint="${arm_prefix_modified}${arm_id}_joint7" transmission="hardware_interface/EffortJointInterface" />
       <xacro:transmission-franka-state arm_id="${arm_id}" />
       <xacro:transmission-franka-model arm_id="${arm_id}"
-         root="${arm_id}_joint1"
-         tip="${arm_id}_joint8"
+         root="${arm_prefix_modified}${arm_id}_joint1"
+         tip="${arm_prefix_modified}${arm_id}_joint8"
        />
       <xacro:if value="${ee_id == 'franka_hand'}">
@@ -162,4 +171,6 @@
           multi_arm="$(arg multi_arm)"
           ee_id="$(arg ee_id)"
+          index="$(arg index)"
+          ns="$(arg ns)"
       />
     </xacro:if>
