Commit message: multirobot_gazebo

File: urdf/franka_arm.ros2_control.xacro (robot description, xacro)
@@ -12,5 +12,5 @@
              multi_arm:=false
              ee_id:=''
-             index:='0'
+             index:=0
              ns:=''
              gripper_closed_position:=0.7929">
@@ -149,7 +149,7 @@
         </gazebo>
       </xacro:unless>
-      <xacro:if value="${multi_arm==1 and index=='0'}">
+      <xacro:if value="${multi_arm==1 and index==0}">
         <gazebo>
-          <plugin filename="ign_ros2_control-system" name="ign_ros2_control::IgnitionROS2ControlPlugin">
+          <plugin filename="gz_ros2_control-system" name="gz_ros2_control::GazeboSimROS2ControlPlugin">
             <parameters>$(find franka_robotiq)/config/multi_franka_gazebo_controllers.yaml</parameters>
           </plugin>

File: urdf/franka_robotiq.xacro (robot description, xacro)
@@ -171,5 +171,5 @@
           multi_arm="$(arg multi_arm)"
           ee_id="$(arg ee_id)"
-          index="$(arg index)"
+          index="${index}"
           ns="$(arg ns)"
       />

File: urdf/multi_arm.urdf.xacro (robot description, xacro)
@@ -44,4 +44,7 @@
   <!-- For a multi arm setup, we need a threaded robot running async-->
   <xacro:arg name="multi_arm" default="true" />
+  <xacro:arg name="ns" default="" />
+  <xacro:arg name="index_arg" default="['0','1']" />
+  <xacro:property name="index_list" value="${$(arg index_arg)}" />
   <!-- Port for gripper communication-->
   <xacro:arg name="com_port" default='/dev/ttyUSB0' />
@@ -70,5 +73,5 @@
       <xacro:arg name="dynamics_path" default="$(find franka_description)/robots/${arm_id_i}/dynamics.yaml"/>
       <xacro:arg name="joint_limits_path" default="$(find franka_description)/robots/${arm_id_i}/joint_limits.yaml"/>
-      <xacro:arg name="index" default="${i}"/>
+      <xacro:property name="index_i" value="${index_list[i]}"/>
       <xacro:franka_robotiq arm_id="${arm_id_i}"
                           joint_limits="${xacro.load_yaml('$(arg joint_limits_path)')}"
@@ -89,5 +92,6 @@
                           connected_to="${arm_prefixes_list[i]}_base"
                           multi_arm="$(arg multi_arm)"
-                          index="$(arg index)">
+                          index="${index_i}"
+                          ns="">
       </xacro:franka_robotiq>
       <xacro:loop i="${i+1}"/>
